File: Kicad_Nb_Iot/NB_Iot_support_TTGO/Support_TTGO/Support_TTGO.kicad_pcb (KiCad board)
At the start: 2 copper layers, 66.9 x 41 mm, 10 parts, among them J1 Conn_01x10, J3 Conn_01x04, J4 Conn_01x04, J5 Conn_01x04, J6 Conn_01x04, J7 Conn_01x03, J8 Conn_01x04

Commit message: update
Parts:
- G***: moved to B.Cu
- moved G*** 1.67 mm to (122.4, 74.5), turned to 90 degrees
Other:
- board text added: "Gnd Clk Data Vcc"
- board text added: "Gnd Data Vcc"
- board text added: "IO_09 IO_10"
- board text added: "IO_09 IO_10 IO_11 IO_12 IO_13 IO_14 Gnd PMU_DC5"
- board text added: "IO_11 IO_12"
- board text added: "IO_13 IO_14"
- board text added: "IO_36 IO_48"
- board text added: "IO_36 IO_48 IO_47 IO_21 Gnd"
- board text added: "IO_47 IO_21"
- board text added: "Temperature DS18B20"
- board text added: "Vcc Data Clk Gnd"
