File: Kicad_Nb_Iot/NB_Iot_support_TTGO/Support_TTGO_Mirroir/Support_TTGO_inversé.kicad_sch (KiCad schematic)
At the start: 9 parts, among them J1 Conn_01x10, J2 Conn_01x10, J3 Conn_01x04, J4 Conn_01x04, J5 Conn_01x04, J6 Conn_01x04, J7 Conn_01x03, J8 Conn_01x04

Commit message: update
Parts:
- added J9: Conn_01x02, Connector_JST:JST_PH_B2B-PH-K_1x02_P2.00mm_Vertical, symbol Connector_Generic:Conn_01x02
- added JP1: SolderJumper_2_Open, Jumper:SolderJumper-2_P1.3mm_Open_RoundedPad1.0x1.5mm, symbol Jumper:SolderJumper_2_Open
- added Q1: PMBT2222A,215, Empreintes:PMBT2222A215, symbol PMBT2222A_215:PMBT2222A,215
- added R2: 4.7k, Resistor_SMD:R_0603_1608Metric, symbol Device:R
Connections:
- net GND: now also Q1.2
- net PMU_DC_DC5: now also JP1.2 (B), R2.1
- net IO_46: now reaches J1.2 (Pin_2)
- net IO_46: now also Q1.1
- new net: J9.2 (Pin_2), JP1.1 (A), R2.2
- new net: J9.1 (Pin_1), Q1.3

Commit message: update
Parts:
- added J10: Conn_01x02, Connector_PinHeader_2.54mm:PinHeader_1x01_P2.54mm_Vertical, symbol Connector_Generic:Conn_01x01
- added J11: Conn_01x02, Connector_JST:JST_PH_B2B-PH-K_1x02_P2.00mm_Vertical, symbol Connector_Generic:Conn_01x02
Connections:
- net GND: now also J3.4 (Pin_4), J4.4 (Pin_4), J5.4 (Pin_4), J6.4 (Pin_4), J7.3 (Pin_3), J8.4 (Pin_4), J11.2 (Pin_2); no longer J3.1 (Pin_1), J4.1 (Pin_1), J5.1 (Pin_1), J6.1 (Pin_1), J7.1 (Pin_1), J8.1 (Pin_1)
- net IO_09: now also J8.3 (Pin_3); no longer J8.2 (Pin_2)
- net IO_10: now also J8.2 (Pin_2); no longer J8.3 (Pin_3)
- net IO_11: now also J4.3 (Pin_3); no longer J4.2 (Pin_2)
- net IO_12: now also J4.2 (Pin_2); no longer J4.3 (Pin_3)
- net IO_13: now also J3.3 (Pin_3); no longer J3.2 (Pin_2)
- net IO_14: now also J3.2 (Pin_2); no longer J3.3 (Pin_3)
- net IO_21: now also J5.3 (Pin_3); no longer J5.2 (Pin_2)
- net IO_36: now also J6.2 (Pin_2); no longer J6.3 (Pin_3)
- net IO_47: now also J5.2 (Pin_2); no longer J5.3 (Pin_3)
- net IO_48: now also J6.3 (Pin_3); no longer J6.2 (Pin_2)
- net PMU_DC_DC5: now also J3.1 (Pin_1), J4.1 (Pin_1), J5.1 (Pin_1), J6.1 (Pin_1), J7.1 (Pin_1), J8.1 (Pin_1); no longer J3.4 (Pin_4), J4.4 (Pin_4), J5.4 (Pin_4), J6.4 (Pin_4), J7.3 (Pin_3), J8.4 (Pin_4)
- net at JP1.1 (A), R2.2: now also J9.1 (Pin_1); no longer J9.2 (Pin_2)
- net at Q1.3: now also J9.2 (Pin_2); no longer J9.1 (Pin_1)
- new net IO_01: J10.1 (Pin_1), J11.1 (Pin_1)
Other:
- moved on the sheet: J5, J6, J7

Commit message: update
Parts:
- removed J6: Conn_01x04, Empreintes:1989764, symbol Connector_Generic:Conn_01x04
- removed JP1: SolderJumper_2_Open, Jumper:SolderJumper-2_P1.3mm_Open_RoundedPad1.0x1.5mm, symbol Jumper:SolderJumper_2_Open
- removed R2: 4.7k, Resistor_SMD:R_0603_1608Metric, symbol Device:R
Connections:
- net IO_21: now also J7.2 (Pin_2), R1.2; no longer J5.3 (Pin_3)
- net IO_47: now also J5.3 (Pin_3); no longer J5.2 (Pin_2)
- net IO_48: now also J5.2 (Pin_2)
- net PMU_DC_DC5: now also J9.1 (Pin_1)
- net IO_01 renamed IO_02
- net IO_36: no longer names the net of J2.2 (Pin_2)
- removed net IO_37: J2.1 (Pin_1), J7.2 (Pin_2), R1.2

Commit message: update
Parts:
- J10: footprint Connector_PinHeader_2.54mm:PinHeader_1x01_P2.54mm_Vertical -> Connector_PinHeader_2.54mm:PinHeader_1x02_P2.54mm_Vertical; symbol Connector_Generic:Conn_01x01 -> Connector_Generic:Conn_01x02
Connections:
- net IO_46: no longer names the net of J1.2 (Pin_2)
- net IO_46: no longer Q1.1
- new net IO_01: J10.2 (Pin_2), Q1.1
Changed lines of the file:
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@@
+    (stroke (width 0) (type default))
+  )
+  (wire (pts (xy 98.552 85.852) (xy 107.442 85.852))
     (stroke (width 0) (type default))
   )
@@
     (stroke (width 0) (type default))
   )
-  (wire (pts (xy 147.066 95.758) (xy 161.036 95.758))
-    (stroke (width 0) (type default))
-  )
   (wire (pts (xy 205.486 70.866) (xy 179.324 70.866))
     (stroke (width 0) (type default))
@@
     )
   )
-  (global_label "IO_46" (shape input) (at 26.162 157.226 180) (fields_autoplaced)
+  (global_label "IO_01" (shape input) (at 26.162 157.226 180) (fields_autoplaced)
     (effects (font (size 1.27 1.27)) (justify right))
     (property "Intersheetrefs" "${INTERSHEET_REFS}" (at 17.9343 157.226 0)
@@
     )
   )
+  (global_label "IO_01" (shape output) (at 98.552 85.852 180) (fields_autoplaced)
+    (effects (font (size 1.27 1.27)) (justify right))
+    (property "Intersheetrefs" "${INTERSHEET_REFS}" (at 90.3243 85.852 0)
+      (effects (font (size 1.27 1.27)) (justify right) hide)
+    )
+  )
   (global_label "PMU_DC_DC5" (shape output) (at 161.036 116.078 0) (fields_autoplaced)
     (effects (font (size 1.27 1.27)) (justify left))
@@
     (effects (font (size 1.27 1.27)) (justify left))
     (property "Intersheetrefs" "${INTERSHEET_REFS}" (at 169.2637 103.378 0)
-      (effects (font (size 1.27 1.27)) (justify left) hide)
-    )
-  )
-  (global_label "IO_46" (shape output) (at 161.036 95.758 0) (fields_autoplaced)
-    (effects (font (size 1.27 1.27)) (justify left))
-    (property "Intersheetrefs" "${INTERSHEET_REFS}" (at 169.2637 95.758 0)
       (effects (font (size 1.27 1.27)) (justify left) hide)
     )
@@
     )
   )
-  (symbol (lib_id "Connector_Generic:Conn_01x01") (at 112.522 83.312 0) (unit 1)
+  (symbol (lib_id "Connector_Generic:Conn_01x02") (at 112.522 83.312 0) (unit 1)
     (in_bom yes) (on_board yes) (dnp no) (fields_autoplaced)
     (property "Reference" "J10" (at 114.554 83.9383 0)
@@
       (effects (font (size 1.27 1.27)) (justify left))
     )
-    (property "Footprint" "Connector_PinHeader_2.54mm:PinHeader_1x01_P2.54mm_Vertical" (at 112.522 83.312 0)
+    (property "Footprint" "Connector_PinHeader_2.54mm:PinHeader_1x02_P2.54mm_Vertical" (at 112.522 83.312 0)
       (effects (font (size 1.27 1.27)) hide)
     )
@@
     )
     (pin "1")
+    (pin "2")
     (instances
       (project "Support_TTGO_inversé"

Commit message: update
Other:
- added sheet HX711 (untitled.kicad_sch)
Changed lines of the file:
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@@
+    )
+  )
+  (sheet (at 312.42 0.508) (size 328.676 209.55)
+    (stroke (width 0.1524) (type solid))
+    (fill (color 0 0 0 0.0000))
+    (property "Sheetname" "HX711" (at 312.928 -1.524 0)
+      (effects (font (size 1.27 1.27)) (justify left bottom))
+    )
+    (property "Sheetfile" "untitled.kicad_sch" (at 312.42 170.0026 0)
+      (effects (font (size 1.27 1.27)) (justify left top))
+    )
+    (instances
+      (project "Support_TTGO_inversé"
+        (path "/ec613b36-6881-4eb0-a769-baf137e1cac3" (page "2"))
+      )
     )
   )
