File: Kicad_Nb_Iot/NB_Iot_support_TTGO/Support_TTGO_Mirroir/Support_TTGO_inversé.kicad_pcb (KiCad board)
At the start: 2 copper layers, 66.9 x 41 mm, 10 parts, among them J1 Conn_01x10, J2 Conn_01x10, J3 Conn_01x04, J4 Conn_01x04, J5 Conn_01x04, J6 Conn_01x04, J7 Conn_01x03, J8 Conn_01x04

Commit message: update
Parts:
- added J9: Conn_01x02, Connector_JST:JST_PH_B2B-PH-K_1x02_P2.00mm_Vertical, F.Cu at (123.6, 70.2)
- added JP1: SolderJumper_2_Open, Jumper:SolderJumper-2_P1.3mm_Open_RoundedPad1.0x1.5mm, B.Cu at (126.1, 74.7)
- added Q1: PMBT2222A,215, Package_TO_SOT_SMD:SOT-23, B.Cu at (120.9, 74.4)
- added R2: 4.7k, Resistor_SMD:R_0603_1608Metric, B.Cu at (124.1, 74.6)
- moved G*** 6.41 mm to (121.7, 80.9)
Connections:
- J1 pad 2: unconnected-(J1-Pin_2-Pad2) -> IO_46
Routing:
- net IO_46: track 0.00 -> 14.4 mm, vias 0 -> 1
- net PMU_DC_DC5: track 130.9 -> 140.5 mm
- net Net-(J9-Pin_2): track 0.00 -> 6.85 mm
- net Net-(J9-Pin_1): track 0.00 -> 5.28 mm
- net GND: vias 0 -> 2
Other:
- outline, holes or cut-outs redrawn
- board text added: "IO_46 IO_09 IO_10 IO_11 IO_12 IO_13 IO_14 Gnd PMU_DC5"
- board text added: "Led"
- board text removed: "IO_09 IO_10 IO_11 IO_12 IO_13 IO_14 Gnd PMU_DC5"
- board text removed: "Vcc=R Data=Y Clk=W Gnd=B"

Commit message: update
Parts:
- added J10: Conn_01x02, Connector_PinHeader_2.54mm:PinHeader_1x01_P2.54mm_Vertical, F.Cu at (156.6, 76.0)
- added J11: locked, Connector_JST:JST_PH_B2B-PH-K_1x02_P2.00mm_Vertical, B.Cu at (159.5, 70.2)
- G***, JP1, Q1, R1, R2: moved to F.Cu
- J3, J4, J5, J6, J7, J8, J9: moved to B.Cu
- moved J5 6.71 mm to (169.0, 98.6), turned to -90 degrees
- moved J6 6.50 mm to (169.0, 85.1), turned to -90 degrees
- moved J8 6.48 mm to (113.7, 78.1), turned to 90 degrees
- moved J7 6.44 mm to (169.0, 71.3), turned to -90 degrees
- moved J4 6.09 mm to (113.7, 91.4), turned to 90 degrees
- moved J3 5.92 mm to (113.6, 105.1), turned to 90 degrees
- moved R1 3.22 mm to (164.2, 77.5), turned to 90 degrees
- moved J9 2.04 mm to (125.6, 70.2), turned to 180 degrees
- moved G*** 1.61 mm to (120.7, 82.1)
- moved Q1 1.32 mm to (121.4, 75.6)
- moved JP1 0.19 mm to (126.2, 74.8)
- moved R2 0.16 mm to (124.1, 74.8)
Connections:
- J3 pad 1: GND -> PMU_DC_DC5
- J3 pad 2: IO_13 -> IO_14
- J3 pad 3: IO_14 -> IO_13
- J3 pad 4: PMU_DC_DC5 -> GND
- J4 pad 1: GND -> PMU_DC_DC5
- J4 pad 2: IO_11 -> IO_12
- J4 pad 3: IO_12 -> IO_11
- J4 pad 4: PMU_DC_DC5 -> GND
- J5 pad 1: GND -> PMU_DC_DC5
- J5 pad 2: IO_21 -> IO_47
- J5 pad 3: IO_47 -> IO_21
- J5 pad 4: PMU_DC_DC5 -> GND
- J6 pad 1: GND -> PMU_DC_DC5
- J6 pad 2: IO_48 -> IO_36
- J6 pad 3: IO_36 -> IO_48
- J6 pad 4: PMU_DC_DC5 -> GND
- J7 pad 1: GND -> PMU_DC_DC5
- J7 pad 3: PMU_DC_DC5 -> GND
- J8 pad 1: GND -> PMU_DC_DC5
- J8 pad 2: IO_09 -> IO_10
- J8 pad 3: IO_10 -> IO_09
- J8 pad 4: PMU_DC_DC5 -> GND
- JP1 pad 1: Net-(J9-Pin_2) -> Net-(J9-Pin_1)
- Q1 pad 3: Net-(J9-Pin_1) -> Net-(J9-Pin_2)
- R2 pad 2: Net-(J9-Pin_2) -> Net-(J9-Pin_1)
Routing:
- net IO_01: track 0.00 -> 7.75 mm
- net Net-(J9-Pin_1): track 5.28 -> 7.12 mm
- net IO_10: track 24.6 -> 23.0 mm
- net IO_46: track 14.4 -> 12.9 mm, vias 1 -> 0
- net Net-(J9-Pin_2): track 6.85 -> 5.37 mm
- net PMU_DC_DC5: track 140.5 -> 141.4 mm, vias 0 -> 2
- net IO_13: track 14.0 -> 13.4 mm
- net IO_14: track 14.0 -> 13.4 mm
- net IO_12: track 15.3 -> 15.8 mm
- net IO_11: track 15.3 -> 15.8 mm
- net GND: vias 2 -> 1
Other:
- board text added: "IO_01"
- board text added: "IO_37"
- board text added: "IO_46 IO_09 IO_10 IO_11 IO_12 IO_13 IO_14 Gnd PMU DC5"
- board text added: "Wifi"
- board text removed: "IO_46 IO_09 IO_10 IO_11 IO_12 IO_13 IO_14 Gnd PMU_DC5"

Commit message: update
Parts:
- removed J6: Conn_01x04, Empreintes:1989764
- removed JP1: SolderJumper_2_Open, Jumper:SolderJumper-2_P1.3mm_Open_RoundedPad1.0x1.5mm
- removed R2: 4.7k, Resistor_SMD:R_0603_1608Metric
- added REF**: PinHeader_1x14_P2.54mm_Vertical, Connector_PinHeader_2.54mm:PinHeader_1x14_P2.54mm_Vertical, F.Cu at (182.4, 70.8)
- moved J7 14.0 mm to (169.0, 85.4)
- moved R1 10.1 mm to (163.6, 87.6), turned to -90 degrees
Connections:
- net IO_01 renamed IO_02
- J2 pad 1: IO_37 -> unconnected-(J2-Pin_1-Pad1)
- J2 pad 2: IO_36 -> unconnected-(J2-Pin_2-Pad2)
- J5 pad 2: IO_47 -> IO_48
- J5 pad 3: IO_21 -> IO_47
- J7 pad 2: IO_37 -> IO_21
- J9 pad 1: Net-(J9-Pin_1) -> PMU_DC_DC5
- R1 pad 2: IO_37 -> IO_21
Routing:
- net IO_37: track 20.6 -> 0.00 mm
- net IO_36: track 12.9 -> 0.00 mm
- net IO_21: track 13.3 -> 26.0 mm, vias 0 -> 1
- net Net-(J9-Pin_1): track 7.12 -> 0.00 mm
- net PMU_DC_DC5: track 141.4 -> 135.9 mm, vias 2 -> 1
- net IO_47: track 13.3 -> 14.3 mm
Other:
- board text added: "IO_21"
- board text removed: "IO_36 IO_48"
- board text removed: "IO_37"

Commit message: update
Parts:
- removed REF**: PinHeader_1x14_P2.54mm_Vertical, Connector_PinHeader_2.54mm:PinHeader_1x14_P2.54mm_Vertical
- added G***: LOGO, Empreintes:Logo Ratamuse petit, B.Cu at (161.4, 79.2)
- added J9: Conn_01x02, Connector_JST:JST_PH_B2B-PH-K_1x02_P2.00mm_Vertical, B.Cu at (172.6, 80.1)
- J10: footprint Connector_PinHeader_2.54mm:PinHeader_1x01_P2.54mm_Vertical -> Connector_PinHeader_2.54mm:PinHeader_1x02_P2.54mm_Vertical
- moved Q1 40.2 mm to (161.6, 75.0), turned to 0 degrees
- moved J9 38.3 mm to (163.8, 70.6)
- moved J11 11.5 mm to (171.0, 70.6)
- moved G*** 7.60 mm to (123.2, 75.0), turned to 80 degrees
- turned J10 to 180 degrees
Connections:
- J1 pad 2: IO_46 -> unconnected-(J1-Pin_2-Pad2)
- Q1 pad 1: IO_46 -> IO_01
Routing:
- net IO_46: track 12.9 -> 0.00 mm
- net IO_02: track 7.75 -> 18.2 mm
- net PMU_DC_DC5: track 135.9 -> 143.0 mm, vias 1 -> 0
- net IO_01: track 0.00 -> 4.31 mm
- net IO_21: track 26.0 -> 24.9 mm
- net Net-(J9-Pin_2): track 5.37 -> 4.70 mm
- net GND: vias 1 -> 0
Other:
- board text added: "IO_48 IO_47"
- board text added: "PB_Pwr"
- board text added: "PB_Wifi"
- board text added: "Scale 1"
- board text added: "Scale 2"
- board text added: "Scale 3"
- board text added: "Scale 4"
- board text added: "Temperature"
- board text removed: "IO_01"
- board text removed: "IO_36 IO_48 IO_47 IO_21 Gnd"
- board text removed: "IO_46 IO_09 IO_10 IO_11 IO_12 IO_13 IO_14 Gnd PMU DC5"
- board text removed: "IO_47 IO_21"
- board text removed: "Temperature DS18B20"
- board text removed: "Wifi"

Commit message: update
Parts:
- added C1: 0.1µF, Capacitor_SMD:C_0603_1608Metric, F.Cu at (215.5, 20.7)
- added C10: 0.1µF, Capacitor_SMD:C_0603_1608Metric, F.Cu at (215.5, 38.3)
- added C11: 0.1µF, Capacitor_SMD:C_0603_1608Metric, F.Cu at (215.5, 40.8)
- added C12: 0.1µF, Capacitor_SMD:C_0603_1608Metric, F.Cu at (219.5, 20.7)
- added C13: 10µF, Capacitor_SMD:C_0805_2012Metric, F.Cu at (198.8, 27.0)
- added C14: 10µF, Capacitor_SMD:C_0805_2012Metric, F.Cu at (198.8, 30.0)
- added C15: 0.1µF, Capacitor_SMD:C_0603_1608Metric, F.Cu at (219.5, 23.2)
- added C16: 0.1µF, Capacitor_SMD:C_0603_1608Metric, F.Cu at (219.5, 25.7)
- added C17: 10µF, Capacitor_SMD:C_0805_2012Metric, F.Cu at (198.8, 33.0)
- added C18: 10µF, Capacitor_SMD:C_0805_2012Metric, F.Cu at (198.8, 36.0)
- added C19: 0.1µF, Capacitor_SMD:C_0603_1608Metric, F.Cu at (219.5, 28.2)
- added C2: 0.1µF, Capacitor_SMD:C_0603_1608Metric, F.Cu at (215.5, 23.2)
- added C20: 0.1µF, Capacitor_SMD:C_0603_1608Metric, F.Cu at (219.5, 30.7)
- added C21: 0.1µF, Capacitor_SMD:C_0603_1608Metric, F.Cu at (219.5, 33.2)
- added C22: 0.1µF, Capacitor_SMD:C_0603_1608Metric, F.Cu at (219.5, 35.8)
- added C23: 0.1µF, Capacitor_SMD:C_0603_1608Metric, F.Cu at (219.5, 38.3)
- added C24: 0.1µF, Capacitor_SMD:C_0603_1608Metric, F.Cu at (219.5, 40.8)
- added C25: 0.1µF, Capacitor_SMD:C_0603_1608Metric, F.Cu at (223.5, 20.7)
- added C26: 0.1µF, Capacitor_SMD:C_0603_1608Metric, F.Cu at (223.5, 23.2)
- added C27: 10µF, Capacitor_SMD:C_0805_2012Metric, F.Cu at (198.8, 39.0)
- added C28: 10µF, Capacitor_SMD:C_0805_2012Metric, F.Cu at (198.8, 42.0)
- added C3: 10µF, Capacitor_SMD:C_0805_2012Metric, F.Cu at (198.8, 20.9)
- added C4: 10µF, Capacitor_SMD:C_0805_2012Metric, F.Cu at (198.8, 23.9)
- added C5: 0.1µF, Capacitor_SMD:C_0603_1608Metric, F.Cu at (215.5, 25.7)
- added C6: 0.1µF, Capacitor_SMD:C_0603_1608Metric, F.Cu at (215.5, 28.2)
- added C7: 0.1µF, Capacitor_SMD:C_0603_1608Metric, F.Cu at (215.5, 30.7)
- added C8: 0.1µF, Capacitor_SMD:C_0603_1608Metric, F.Cu at (215.5, 33.2)
- added C9: 0.1µF, Capacitor_SMD:C_0603_1608Metric, F.Cu at (215.5, 35.8)
- added J12: Conn_01x02, Empreintes:SHDR2W90P0X500_1X2_1060X980X1380P, F.Cu at (204.3, 25.4)
- added J16: Conn_01x02, Empreintes:SHDR2W90P0X500_1X2_1060X980X1380P, F.Cu at (204.3, 36.8)
- added L1: 3.3µH, Inductor_SMD:L_0603_1608Metric, F.Cu at (223.5, 25.7)
- added L2: 3.3µH, Inductor_SMD:L_0603_1608Metric, F.Cu at (223.5, 28.2)
- added L3: 3.3µH, Inductor_SMD:L_0603_1608Metric, F.Cu at (223.5, 30.7)
- added L4: 3.3µH, Inductor_SMD:L_0603_1608Metric, F.Cu at (223.5, 33.2)
- added Q2: MMBT4403, Package_TO_SOT_SMD:SOT-23, F.Cu at (215.9, 44.2)
- added Q3: MMBT4403, Package_TO_SOT_SMD:SOT-23, F.Cu at (215.9, 48.7)
- added Q4: MMBT4403, Package_TO_SOT_SMD:SOT-23, F.Cu at (215.9, 53.1)
- added Q5: MMBT4403, Package_TO_SOT_SMD:SOT-23, F.Cu at (215.9, 57.6)
- added R10: 20K, Resistor_SMD:R_0603_1608Metric, F.Cu at (227.5, 33.2)
- added R11: 8.2K, Resistor_SMD:R_0603_1608Metric, F.Cu at (227.5, 35.8)
- added R12: 100, Resistor_SMD:R_0603_1608Metric, F.Cu at (227.5, 38.3)
- added R13: 100, Resistor_SMD:R_0603_1608Metric, F.Cu at (227.5, 40.8)
- added R14: 20K, Resistor_SMD:R_0603_1608Metric, F.Cu at (231.5, 20.7)
- added R15: 8.2K, Resistor_SMD:R_0603_1608Metric, F.Cu at (231.5, 23.2)
- added R16: 100, Resistor_SMD:R_0603_1608Metric, F.Cu at (231.5, 25.7)
- added R17: 100, Resistor_SMD:R_0603_1608Metric, F.Cu at (231.5, 28.2)
- added R2: 20K, Resistor_SMD:R_0603_1608Metric, F.Cu at (223.5, 35.8)
- added R3: 8.2K, Resistor_SMD:R_0603_1608Metric, F.Cu at (223.5, 38.3)
- added R4: 100, Resistor_SMD:R_0603_1608Metric, F.Cu at (223.5, 40.8)
- added R5: 100, Resistor_SMD:R_0603_1608Metric, F.Cu at (227.5, 20.7)
- added R6: 20K, Resistor_SMD:R_0603_1608Metric, F.Cu at (227.5, 23.2)
- added R7: 8.2K, Resistor_SMD:R_0603_1608Metric, F.Cu at (227.5, 25.7)
- added R8: 100, Resistor_SMD:R_0603_1608Metric, F.Cu at (227.5, 28.2)
- added R9: 100, Resistor_SMD:R_0603_1608Metric, F.Cu at (227.5, 30.7)
Connections:
- J9 pad 1: GND -> PMU_DC_DC5
- J9 pad 2: (no net) -> Net-(J9-Pin_2)
